Commit message: multi kim sol

File: basic134/urdf/example.urdf (robot description, URDF)
Before this commit: robot example, 9 links, 8 joints
Links:
- link lbracket: geometry visual mesh filename=package://basic134/meshes/Lbracket.stl scale=1.0 1.0 1.0
Joints:
- removed joint base
- removed joint elbow
- removed joint shoulder
- added joint theta1: type continuous, parent basemotor, child lbracket, origin xyz=0 0 0.0311 rpy=0 0 1.5708, axis 0 0 1
- added joint theta2: type continuous, parent shouldermotor, child upperarm, origin xyz=0 0 0.0451 rpy=0 0 -1.5708, axis 0 0 1
- added joint theta3: type continuous, parent elbowmotor, child lowerarm, origin xyz=0 0 0.0311 rpy=0 0 0, axis 0 0 1
- joint lbracket: origin xyz=0.1 0 0.1 rpy=1.5708 0 -1.5708 -> xyz=0.075 0 0.065625 rpy=1.5708 1.5708 -1.5708

Commit message: floating

File: basic134/urdf/example.urdf (robot description, URDF)
Before this commit: robot example, 9 links, 8 joints
Links:
- link lowerarm: geometry visual mesh filename=package://basic134/meshes/arm_tip.stl scale=0.001 0.001 0.001
- link upperarm: geometry visual mesh filename=package://basic134/meshes/arm.stl scale=0.001 0.001 0.001
Joints:
- joint lbracket: origin xyz=0.075 0 0.065625 rpy=1.5708 1.5708 -1.5708 -> xyz=0.0450 0 0.078 rpy=1.5708 1.5708 -1.5708

Commit message: grap sth

File: basic134/urdf/example.urdf (robot description, URDF)
Before this commit: robot example, 9 links, 8 joints
Joints:
- joint lowerarm: origin xyz=0.5 0 0.003175 rpy=0 0 0 -> xyz=0.5 0 0.003175 rpy=0 0 0.7854
