Commit message: gripper stl

File: sixdof/urdf/example.urdf (robot description, URDF)
Before this commit: robot example, 13 links, 12 joints
Links:
- link tip: geometry visual mesh filename=package://basic134/meshes/gripper.stl scale=0.005 0.005 0.005
Joints:
- joint finger: origin xyz=0 0 0.09 rpy=0 0 0 -> xyz=0 0 0.09 rpy=0 0 0.7854

Commit message: flip skeleton

File: sixdof/urdf/example.urdf (robot description, URDF)
Before this commit: robot example, 13 links, 12 joints
Joints:
- joint theta1: origin xyz=0 0 0.0311 rpy=0 0 1.5708 -> xyz=0 0 0.0451 rpy=0 0 1.5708

Commit message: err fix

File: sixdof/urdf/example.urdf (robot description, URDF)
Before this commit: robot example, 13 links, 12 joints
Links:
- link basemotor: geometry visual mesh filename=package://basic134/meshes/X8.stl scale=0.001 0.001 0.001
- link palm: geometry visual mesh filename=package://basic134/meshes/wrist_Lbracket.stl scale=0.001 0.001 0.001
- link tip: geometry visual mesh filename=package://basic134/meshes/gripper_tips.stl scale=0.001 0.001 0.001
Joints:
- joint finger: origin xyz=0 0 0.09 rpy=0 0 0.7854 -> xyz=0 0 0.105 rpy=0 0 0.7854
- joint theta1: origin xyz=0 0 0.0451 rpy=0 0 1.5708 -> xyz=0 0 0.045 rpy=0 0 1.5708
- joint theta2: origin xyz=0 0 0.0451 rpy=0 0 -1.5708 -> xyz=0 0 0.05 rpy=0 0 -1.5708
- joint theta3: origin xyz=0 0 0.0311 rpy=0 0 0 -> xyz=0 0 0.031 rpy=0 0 0
- joint theta5: origin xyz=0 0 0.0311 rpy=0 0 0 -> xyz=0 0 0.031 rpy=0 0 0
- joint upperarm: origin xyz=0.395 0 0.0127 rpy=0 0 0 -> xyz=0.395 0 0.01 rpy=0 0 0
